File: kicad/$protoBaguette.sch (KiCad schematic (older format))
At the start: 42 parts, among them J1 RJ45-MAG, P1 HEADER_5, P2 HEADER_4, P3 HEADER_5, P4 HEADER_5, U1 NX1117C, U2 PIC32MX150F128-1, U3 ENC28J60-1, X1 CRYSTAL

Commit message: Final layout, before footprint inspection
Parts:
- C8: value 100n? -> 10u
Changed lines of the file:
@@
-EESchema Schematic File Version 2  date dim. 09 juin 2013 16:16:57 CEST
+EESchema Schematic File Version 2  date dim. 09 juin 2013 18:51:20 CEST
 LIBS:power
 LIBS:device
@@
 encoding utf-8
 Sheet 1 1
-Title "Alpha prototype"
+Title "ProtoBaguette, first board"
 Date "9 jun 2013"
-Rev "0.1"
-Comp "ProtoBaguette"
+Rev "1.0"
+Comp "Hexabread"
 Comment1 ""
 Comment2 ""
@@
 	1850 3200 650  3200
 $Comp
-L GND #PWR?
+L GND #PWR01
 U 1 1 51B48E51
 P 1400 2850
-F 0 "#PWR?" H 1400 2850 30  0001 C CNN
+F 0 "#PWR01" H 1400 2850 30  0001 C CNN
 F 1 "GND" H 1400 2780 30  0001 C CNN
 	1    1400 2850
@@
 $EndComp
 $Comp
-L VDD #PWR3
+L VDD #PWR02
 U 1 1 51B47A9A
 P 1350 3350
-F 0 "#PWR3" H 1350 3450 30  0001 C CNN
+F 0 "#PWR02" H 1350 3450 30  0001 C CNN
 F 1 "VDD" H 1350 3460 30  0000 C CNN
 	1    1350 3350
@@
 BO6
 $Comp
-L VDD #PWR15
+L VDD #PWR03
 U 1 1 51B46A29
 P 3700 2100
-F 0 "#PWR15" H 3700 2200 30  0001 C CNN
+F 0 "#PWR03" H 3700 2200 30  0001 C CNN
 F 1 "VDD" H 3700 2210 30  0000 C CNN
 	1    3700 2100
@@
 $EndComp
 $Comp
-L VDD #PWR12
+L VDD #PWR04
 U 1 1 51B46230
 P 2750 800
-F 0 "#PWR12" H 2750 900 30  0001 C CNN
+F 0 "#PWR04" H 2750 900 30  0001 C CNN
 F 1 "VDD" H 2750 910 30  0000 C CNN
 	1    2750 800
@@
 $EndComp
 $Comp
-L GND #PWR22
+L GND #PWR05
 U 1 1 51B331B8
 P 7900 5450
-F 0 "#PWR22" H 7900 5450 30  0001 C CNN
+F 0 "#PWR05" H 7900 5450 30  0001 C CNN
 F 1 "GND" H 7900 5380 30  0001 C CNN
 	1    7900 5450
@@
 $EndComp
 $Comp
-L VDD #PWR8
+L VDD #PWR06
 U 1 1 51B32F4B
 P 2250 3800
-F 0 "#PWR8" H 2250 3900 30  0001 C CNN
+F 0 "#PWR06" H 2250 3900 30  0001 C CNN
 F 1 "VDD" H 2250 3910 30  0000 C CNN
 	1    2250 3800
@@
 NoConn ~ 4050 6700
 $Comp
-L GND #PWR16
+L GND #PWR07
 U 1 1 51B3216A
 P 4050 6900
-F 0 "#PWR16" H 4050 6900 30  0001 C CNN
+F 0 "#PWR07" H 4050 6900 30  0001 C CNN
 F 1 "GND" H 4050 6830 30  0001 C CNN
 	1    4050 6900
@@
 $EndComp
 $Comp
-L VDD #PWR18
+L VDD #PWR08
 U 1 1 51B312CD
 P 4850 950
-F 0 "#PWR18" H 4850 1050 30  0001 C CNN
+F 0 "#PWR08" H 4850 1050 30  0001 C CNN
 F 1 "VDD" H 4850 1060 30  0000 C CNN
 	1    4850 950
@@
 $EndComp
 $Comp
-L GND #PWR17
+L GND #PWR09
 U 1 1 51B312CC
 P 4200 1650
-F 0 "#PWR17" H 4200 1650 30  0001 C CNN
+F 0 "#PWR09" H 4200 1650 30  0001 C CNN
 F 1 "GND" H 4200 1580 30  0001 C CNN
 	1    4200 1650
@@
 P 7500 1250
 F 0 "C8" H 7550 1350 50  0000 L CNN
-F 1 "100n?" H 7550 1150 50  0000 L CNN
+F 1 "10u" H 7550 1150 50  0000 L CNN
 	1    7500 1250
 	1    0    0    -1
@@
 $EndComp
 $Comp
-L GND #PWR14
+L GND #PWR010
 U 1 1 51AB2611
 P 3350 3900
-F 0 "#PWR14" H 3350 3900 30  0001 C CNN
+F 0 "#PWR010" H 3350 3900 30  0001 C CNN
 F 1 "GND" H 3350 3830 30  0001 C CNN
 	1    3350 3900
@@
 $EndComp
 $Comp
-L VDD #PWR13
+L VDD #PWR011
 U 1 1 51AB2265
 P 3250 3300
-F 0 "#PWR13" H 3250 3400 30  0001 C CNN
+F 0 "#PWR011" H 3250 3400 30  0001 C CNN
 F 1 "VDD" H 3250 3410 30  0000 C CNN
 	1    3250 3300
@@
 $EndComp
 $Comp
-L GND #PWR23
+L GND #PWR012
 U 1 1 519A8426
 P 9150 5150
-F 0 "#PWR23" H 9150 5150 30  0001 C CNN
+F 0 "#PWR012" H 9150 5150 30  0001 C CNN
 F 1 "GND" H 9150 5080 30  0001 C CNN
 	1    9150 5150
@@
 Microchip ICSP
 $Comp
-L VDD #PWR4
+L VDD #PWR013
 U 1 1 519A81F2
 P 1400 2150
-F 0 "#PWR4" H 1400 2250 30  0001 C CNN
+F 0 "#PWR013" H 1400 2250 30  0001 C CNN
 F 1 "VDD" H 1400 2260 30  0000 C CNN
 	1    1400 2150
@@
 $EndComp
 $Comp
-L GND #PWR1
+L GND #PWR014
 U 1 1 519A80F8
 P 1300 4450
-F 0 "#PWR1" H 1300 4450 30  0001 C CNN
+F 0 "#PWR014" H 1300 4450 30  0001 C CNN
 F 1 "GND" H 1300 4380 30  0001 C CNN
 	1    1300 4450
@@
 User ETHERNET SOCKET
 $Comp
-L GND #PWR9
+L GND #PWR015
 U 1 1 519A7550
 P 2300 6450
-F 0 "#PWR9" H 2300 6450 30  0001 C CNN
+F 0 "#PWR015" H 2300 6450 30  0001 C CNN
 F 1 "GND" H 2300 6380 30  0001 C CNN
 	1    2300 6450
@@
 LEDA
 $Comp
-L GND #PWR11
+L GND #PWR016
 U 1 1 519A74FC
 P 2300 6850
-F 0 "#PWR11" H 2300 6850 30  0001 C CNN
+F 0 "#PWR016" H 2300 6850 30  0001 C CNN
 F 1 "GND" H 2300 6780 30  0001 C CNN
 	1    2300 6850
@@
 $EndComp
 $Comp
-L GND #PWR10
+L GND #PWR017
 U 1 1 519A74EF
 P 2300 6650
-F 0 "#PWR10" H 2300 6650 30  0001 C CNN
+F 0 "#PWR017" H 2300 6650 30  0001 C CNN
 F 1 "GND" H 2300 6580 30  0001 C CNN
 	1    2300 6650
@@
 $EndComp
 $Comp
-L GND #PWR7
+L GND #PWR018
 U 1 1 519A737B
 P 2100 7500
-F 0 "#PWR7" H 2100 7500 30  0001 C CNN
+F 0 "#PWR018" H 2100 7500 30  0001 C CNN
 F 1 "GND" H 2100 7430 30  0001 C CNN
 	1    2100 7500
@@
 $EndComp
 $Comp
-L VDD #PWR6
+L VDD #PWR019
 U 1 1 519A7084
 P 2100 5200
-F 0 "#PWR6" H 2100 5300 30  0001 C CNN
+F 0 "#PWR019" H 2100 5300 30  0001 C CNN
 F 1 "VDD" H 2100 5310 30  0000 C CNN
 	1    2100 5200
@@
 $EndComp
 $Comp
-L GND #PWR5
+L GND #PWR020
 U 1 1 519A7081
 P 1750 7500
-F 0 "#PWR5" H 1750 7500 30  0001 C CNN
+F 0 "#PWR020" H 1750 7500 30  0001 C CNN
 F 1 "GND" H 1750 7430 30  0001 C CNN
 	1    1750 7500
@@
 $EndComp
 $Comp
-L VDD #PWR25
+L VDD #PWR021
 U 1 1 519A6DA9
 P 9750 950
-F 0 "#PWR25" H 9750 1050 30  0001 C CNN
+F 0 "#PWR021" H 9750 1050 30  0001 C CNN
 F 1 "VDD" H 9750 1060 30  0000 C CNN
 	1    9750 950
@@
 $EndComp
 $Comp
-L GND #PWR26
+L GND #PWR022
 U 1 1 519A6DA8
 P 9750 1600
-F 0 "#PWR26" H 9750 1600 30  0001 C CNN
+F 0 "#PWR022" H 9750 1600 30  0001 C CNN
 F 1 "GND" H 9750 1530 30  0001 C CNN
 	1    9750 1600
@@
 TPO-
 $Comp
-L GND #PWR21
+L GND #PWR023
 U 1 1 519A6BF7
 P 7100 5200
-F 0 "#PWR21" H 7100 5200 30  0001 C CNN
+F 0 "#PWR023" H 7100 5200 30  0001 C CNN
 F 1 "GND" H 7100 5130 30  0001 C CNN
 	1    7100 5200
@@
 $EndComp
 $Comp
-L VDD #PWR24
+L VDD #PWR024
 U 1 1 519A6BE5
 P 9200 2250
-F 0 "#PWR24" H 9200 2350 30  0001 C CNN
+F 0 "#PWR024" H 9200 2350 30  0001 C CNN
 F 1 "VDD" H 9200 2360 30  0000 C CNN
 	1    9200 2250
@@
 Must be placed near pins
 $Comp
-L GND #PWR20
+L GND #PWR025
 U 1 1 519A6ADD
 P 6150 1550
-F 0 "#PWR20" H 6150 1550 30  0001 C CNN
+F 0 "#PWR025" H 6150 1550 30  0001 C CNN
 F 1 "GND" H 6150 1480 30  0001 C CNN
 	1    6150 1550
@@
 $EndComp
 $Comp
-L VDD #PWR19
+L VDD #PWR026
 U 1 1 519A6AD8
 P 6150 950
-F 0 "#PWR19" H 6150 1050 30  0001 C CNN
+F 0 "#PWR026" H 6150 1050 30  0001 C CNN
 F 1 "VDD" H 6150 1060 30  0000 C CNN
 	1    6150 950
@@
 User UART + POWER
 $Comp
-L GND #PWR2
+L GND #PWR027
 U 1 1 519A6988
 P 1350 1600
-F 0 "#PWR2" H 1350 1600 30  0001 C CNN
+F 0 "#PWR027" H 1350 1600 30  0001 C CNN
 F 1 "GND" H 1350 1530 30  0001 C CNN
 	1    1350 1600
